File: hardware/LoRa_Receiver_Board_REV1/GroundStation_3.kicad_pcb (KiCad board)
At the start: 2 copper layers, 100 x 70 mm, 143 parts, among them IC1 XC8114AA01PR-G, IC2 TBD62384AFWG, J2 USB_B, Q1 BSS138, Q10 BSS138, Q11 BSS138, Q12 BSS138, Q13 BSS84, Q14 BSS84, Q2 BSS138, Q3 BSS138, Q4 BSS138, Q5 BSS138, Q6 BSS138, Q7 BSS138, Q8 BSS138, Q9 BSS138, SW1 PTS645SK50SMTR92LFS, SW2 PTS645SK50SMTR92LFS, U1 ADP151AUJZ-3.3, U10 DG4053EEQ-T1-GE3, U11 ADP3338AKCZ-3.3, U13 DG4053EEQ-T1-GE3, U2 FT4233HPQ-REEL, U3 93LCxxB, U4 ADP151AUJZ-3.3, U5 E22-900T30D_E220-900T22S(JP)_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, U6 E22-900T30D_E220-900T22S(JP)_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, U7 E22-900T30D_E220-900T22S(JP)_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, U8 SAM-M10Q-00B, U9 USBLC6-2SC6, Y1 FA-238V_12.0000MA-C5

Commit message: Update schematic and pcb
Parts:
- removed F3: 0805L100WR, Fuse:Fuse_0805_2012Metric
- removed Q1, Q10, Q11, Q12, Q2, Q3, Q4, Q5, Q6, Q8, Q9: BSS138, Package_TO_SOT_SMD:SOT-23
- removed Q13, Q14: BSS84, Package_TO_SOT_SMD:SOT-23
- removed R1: 1M, Resistor_SMD:R_0603_1608Metric_Pad0.98x0.95mm_HandSolder
- added C41: 0.1u, Capacitor_SMD:C_0603_1608Metric_Pad1.08x0.95mm_HandSolder, B.Cu at (131.2, 70.4)
- added C42: 0.1u, Capacitor_SMD:C_0603_1608Metric_Pad1.08x0.95mm_HandSolder, B.Cu at (138.3, 72.4)
- added C43: 0.1u, Capacitor_SMD:C_0603_1608Metric_Pad1.08x0.95mm_HandSolder, B.Cu at (153.9, 58.7)
- added D17: LED_Small, LED_SMD:LED_0603_1608Metric_Pad1.05x0.95mm_HandSolder, F.Cu at (129.8, 100.5)
- added D18: LED_Small, LED_SMD:LED_0603_1608Metric_Pad1.05x0.95mm_HandSolder, F.Cu at (131.4, 100.5)
- added R37: 1k, Resistor_SMD:R_0603_1608Metric_Pad0.98x0.95mm_HandSolder, B.Cu at (129.8, 102.2)
- added R38: 1k, Resistor_SMD:R_0603_1608Metric_Pad0.98x0.95mm_HandSolder, B.Cu at (131.4, 102.2)
- added R39: 15k, Resistor_SMD:R_0603_1608Metric_Pad0.98x0.95mm_HandSolder, F.Cu at (153.5, 111.8)
- added R40: 100k, Resistor_SMD:R_0603_1608Metric_Pad0.98x0.95mm_HandSolder, F.Cu at (153.5, 110.2)
- C22, C23, C24, C25, C28, C32, C34, C35, C36, C37, C38, C39, D1, D3, IC2, R13, R14, R16, R17, R18, R19, R20, R21, R22, R23, R24, R26, R27, R28, R29, R30, R31, R32, R33, R34, R35, R36, R51, U1, U10, U11, U13: moved to B.Cu
- C3, C4: value 10p -> 27p（C0G/NP0）
- Q7: value BSS138 -> TBD62083AFWG; footprint Package_TO_SOT_SMD:SOT-23 -> Package_SO:SOIC-18W_7.5x11.6mm_P1.27mm; moved to B.Cu
- U4: value ADP151AUJZ-3.3 -> SN74HCT245PWR; footprint Package_TO_SOT_SMD:TSOT-23-5 -> Package_SO:TSSOP-20_4.4x6.5mm_P0.65mm; moved to B.Cu
- moved S1 206.9 mm to (217.3, 65.3), turned to -90 degrees
- moved S2 194.0 mm to (217.3, 77.1), turned to -90 degrees
- moved R16 188.2 mm to (213.8, 68.3)
- moved S3 183.2 mm to (217.3, 89.4), turned to -90 degrees
- moved R20 172.9 mm to (213.8, 86.3), turned to 180 degrees
- moved S4 172.9 mm to (217.3, 101.6), turned to -90 degrees
- moved R17 172.4 mm to (213.8, 80.2), turned to 180 degrees
- moved S5 172.0 mm to (217.3, 83.2), turned to -90 degrees
- moved C34 169.3 mm to (201.8, 87.9)
- moved R21 168.7 mm to (213.8, 98.5), turned to 180 degrees
- moved R18 168.3 mm to (214.0, 92.5), turned to 180 degrees
- moved R22 165.1 mm to (213.8, 110.7), turned to 180 degrees
- moved D1 165.0 mm to (184.5, 70.6)
- moved R19 164.9 mm to (214.2, 104.8), turned to 180 degrees
- moved U13 164.3 mm to (201.5, 72.1)
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Connections:
- D16 pad 2: Net-(D16-A) -> VBUS
- IC2 pad 1: unconnected-(IC2-I1-Pad1) -> Net-(IC2-I1)
- IC2 pad 10: unconnected-(IC2-VCC-Pad10) -> VBUS
- IC2 pad 13: unconnected-(IC2-O6-Pad13) -> Net-(IC2-O6)
- IC2 pad 14: unconnected-(IC2-O5-Pad14) -> Net-(IC2-O5)
- IC2 pad 15: unconnected-(IC2-O4-Pad15) -> Net-(IC2-O4)
- IC2 pad 16: unconnected-(IC2-O3-Pad16) -> Net-(IC2-O3)
- IC2 pad 17: unconnected-(IC2-O2-Pad17) -> Net-(IC2-O2)
- IC2 pad 18: unconnected-(IC2-O1-Pad18) -> Net-(IC2-O1)
- IC2 pad 2: unconnected-(IC2-I2-Pad2) -> Net-(IC2-I2)
- IC2 pad 3: unconnected-(IC2-I3-Pad3) -> Net-(IC2-I3)
- IC2 pad 4: unconnected-(IC2-I4-Pad4) -> Net-(IC2-I4)
- IC2 pad 5: unconnected-(IC2-I5-Pad5) -> Net-(IC2-I5)
- IC2 pad 6: unconnected-(IC2-I6-Pad6) -> Net-(IC2-I6)
- IC2 pad 9: unconnected-(IC2-GND-Pad9) -> GND
- Q7 pad 1: unconnected-(Q7-G-Pad1) -> /LORA_A_M0
- Q7 pad 2: GND -> /LORA_A_M1
- Q7 pad 3: Net-(Q7-D) -> /LORA_B_M0
- R27 pad 1: Net-(Q1-D) -> Net-(Q7-O1)
- R28 pad 1: Net-(Q2-D) -> Net-(Q7-O2)
- R29 pad 1: Net-(Q3-D) -> Net-(Q7-O3)
- R30 pad 1: Net-(Q4-D) -> Net-(Q7-O4)
- R31 pad 1: Net-(Q5-D) -> Net-(Q7-O5)
- R32 pad 1: Net-(Q6-D) -> Net-(Q7-O6)
- R33 pad 1: Net-(Q7-D) -> Net-(IC2-O1)
- R34 pad 1: Net-(Q10-D) -> Net-(IC2-O2)
- R35 pad 1: Net-(Q11-D) -> Net-(IC2-O3)
- R36 pad 1: GND -> Net-(IC2-O4)
- U4 pad 2: GND -> /UART_A_MISO
- U4 pad 3: VBUS -> /UART_A_MOSI
- U4 pad 4: unconnected-(U4-NC-Pad4) -> /UART_B_MISO
- U4 pad 5: +3V3 -> /UART_B_MOSI
Routing:
- net /USB_DM: track 0.00 -> 27.5 mm
- net /USB_DP: track 0.00 -> 27.4 mm
- net Net-(U2-OSCO): track 0.00 -> 9.68 mm
- net Net-(U2-OSCI): track 0.00 -> 6.54 mm
Other:
- copper layers 2 -> 4
- board text added: "LoRa Ground Station Designed by Unknown 2026.11.01 REV2"
