File: hardware/LoRa_Receiver_Board_REV1/GroundStation_3.kicad_sch (KiCad schematic)
At the start: 134 parts, among them IC1 XC8114AA01PR-G, IC2 TBD62384AFWG, J2 USB_B, Q7 TBD62083AFWG, SW1 PTS645SK50SMTR92LFS, SW2 PTS645SK50SMTR92LFS, U1 ADP151AUJZ-3.3, U10 DG4053EEQ-T1-GE3, U11 ADP3338AKCZ-3.3, U13 DG4053EEQ-T1-GE3, U2 FT4233HPQ-REEL, U3 93LCxxB, U5 E22-900T30D_E220-900T22S(JP)_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, U6 E22-900T30D_E220-900T22S(JP)_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, U7 E22-900T30D_E220-900T22S(JP)_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, U8 SAM-M10Q-00B, U9 USBLC6-2SC6, Y1 FA-238V_12.0000MA-C5

Commit message: Update schematic and pcb
Parts:
- removed R1: 1M, Resistor_SMD:R_0603_1608Metric_Pad0.98x0.95mm_HandSolder, symbol Device:R_Small
- added C43: 0.1u, Capacitor_SMD:C_0603_1608Metric_Pad1.08x0.95mm_HandSolder, symbol Device:C_Small
- added R39: 15k, Resistor_SMD:R_0603_1608Metric_Pad0.98x0.95mm_HandSolder, symbol Device:R_Small
- added R40: 100k, Resistor_SMD:R_0603_1608Metric_Pad0.98x0.95mm_HandSolder, symbol Device:R_Small
- added U4: SN74HCT245PWR, Package_SO:TSSOP-20_4.4x6.5mm_P0.65mm, symbol Unknown:SN74HCT245PWR
- C3, C4: value 10p -> 27p（C0G/NP0）
Connections:
- net +3V3: no longer C41.1, C42.1, IC2.10 (VCC), Q7.10 (COMMON)
- net GND: now also C43.2, R39.2, U4.10 (GND), U4.19 (~{OE}), U4.8 (A7), U4.9 (A8)
- net UART_A_MISO: now also U4.2 (A1); no longer IC2.1 (I1)
- net UART_A_MOSI: now also U4.3 (A2); no longer IC2.2 (I2)
- net UART_B_MISO: now also U4.4 (A3); no longer IC2.3 (I3)
- net UART_B_MOSI: now also U4.5 (A4); no longer IC2.4 (I4)
- net UART_C_MISO: now also U4.6 (A5); no longer IC2.5 (I5)
- net UART_C_MOSI: now also U4.7 (A6); no longer IC2.6 (I6)
- net VBUS: now also C41.1, C42.1, IC2.10 (VCC), Q7.10 (COMMON), C43.1, R40.1, U4.1 (DIR), U4.20 (VCC)
- net at U2.68 (PD1_SVBUS): now also R39.1, R40.2
- new net: IC2.6 (I6), U4.13 (B6)
- new net: IC2.5 (I5), U4.14 (B5)
- new net: IC2.4 (I4), U4.15 (B4)
- new net: IC2.3 (I3), U4.16 (B3)
- new net: IC2.2 (I2), U4.17 (B2)
- new net: IC2.1 (I1), U4.18 (B1)
- no-connect marks 29 -> 31
Other:
- note added: "8ch Bus トランシーバー(レベルシフタ) + 8ch Dチャネルトランジスタアレイ（ローアクティブタイプ）"
- note removed: "8ch Dチャネルトランジスタアレイ（ローアクティブタイプ）"
- moved on the sheet: C41, C42, D10, D11, D12, D13, D14, D15, D16, D17, D18, D2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
